File: PCB/main/chu_arcade.kicad_sch (KiCad schematic)
At the start: 44 parts, among them J1 LED_In, J2 LED_Out, J3 Conn_01x04, U2 PCA9548APW, X1 GP2Y0E03_REAL, X2 GP2Y0E03_REAL, X3 GP2Y0E03_REAL, X4 GP2Y0E03_REAL, X5 GP2Y0E03_REAL, X6 GP2Y0E03_REAL

Commit message: Add I2C main pull-up resistors
Parts:
- added R13, R14: 4.7K, Resistor_SMD:R_0603_1608Metric, symbol Device:R_Small
Connections:
- net +3V3: now also R13.1, R14.1
- net SCL: now also R13.2
- net SDA: now also R14.2
Changed lines of the file:
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@@
+    (stroke (width 0) (type default))
+  )
+  (wire (pts (xy 244.475 80.01) (xy 244.475 82.55))
     (stroke (width 0) (type default))
   )
@@
     (stroke (width 0) (type default))
   )
-  (wire (pts (xy 244.475 80.01) (xy 244.475 82.55))
-    (stroke (width 0) (type default))
-  )
   (wire (pts (xy 257.81 97.155) (xy 262.89 97.155))
     (stroke (width 0) (type default))
@@
     (stroke (width 0) (type default))
   )
+  (wire (pts (xy 227.33 82.55) (xy 233.68 82.55))
+    (stroke (width 0) (type default))
+  )
   (wire (pts (xy 200.66 189.23) (xy 213.36 189.23))
     (stroke (width 0) (type default))
@@
     (stroke (width 0) (type default))
   )
+  (wire (pts (xy 238.76 80.01) (xy 244.475 80.01))
+    (stroke (width 0) (type default))
+  )
   (wire (pts (xy 244.475 97.155) (xy 244.475 99.695))
     (stroke (width 0) (type default))
@@
     (stroke (width 0) (type default))
   )
+  (wire (pts (xy 227.33 80.01) (xy 233.68 80.01))
+    (stroke (width 0) (type default))
+  )
   (wire (pts (xy 257.175 114.3) (xy 262.89 114.3))
     (stroke (width 0) (type default))
@@
     (stroke (width 0) (type default))
   )
+  (wire (pts (xy 244.475 74.93) (xy 244.475 77.47))
+    (stroke (width 0) (type default))
+  )
   (wire (pts (xy 201.93 86.995) (xy 201.93 88.9))
     (stroke (width 0) (type default))
@@
     (stroke (width 0) (type default))
   )
+  (wire (pts (xy 238.76 82.55) (xy 244.475 82.55))
+    (stroke (width 0) (type default))
+  )
   (wire (pts (xy 137.16 200.66) (xy 149.86 200.66))
-    (stroke (width 0) (type default))
-  )
-  (wire (pts (xy 244.475 74.93) (xy 244.475 77.47))
     (stroke (width 0) (type default))
   )
@@
     (effects (font (size 1 1)) (justify left bottom))
   )
+  (label "SCL" (at 227.33 80.01 180) (fields_autoplaced)
+    (effects (font (size 1 1)) (justify right bottom))
+  )
   (label "SCL_2" (at 212.09 120.65 0) (fields_autoplaced)
     (effects (font (size 1 1)) (justify left bottom))
@@
   )
   (label "SDA_1" (at 262.89 82.55 180) (fields_autoplaced)
+    (effects (font (size 1 1)) (justify right bottom))
+  )
+  (label "SDA" (at 227.33 82.55 180) (fields_autoplaced)
     (effects (font (size 1 1)) (justify right bottom))
   )
@@
     )
   )
+  (symbol (lib_id "Device:R_Small") (at 236.22 80.01 270) (unit 1)
+    (in_bom yes) (on_board yes) (dnp no)
+    (property "Reference" "R13" (at 229.87 78.74 90)
+      (effects (font (size 1.27 1.27)) (justify left))
+    )
+    (property "Value" "4.7K" (at 234.7888 80.0382 90)
+      (effects (font (size 0.8 0.8)) (justify left))
+    )
+    (property "Footprint" "Resistor_SMD:R_0603_1608Metric" (at 236.22 80.01 0)
+      (effects (font (size 1.27 1.27)) hide)
+    )
+    (property "Datasheet" "~" (at 236.22 80.01 0)
+      (effects (font (size 1.27 1.27)) hide)
+    )
+    (property "LCSC" "C23186" (at 236.22 80.01 0)
+      (effects (font (size 1.27 1.27)) hide)
+    )
+    (pin "1")
+    (pin "2")
+    (instances
+      (project "chu_arcade"
+        (path "/2e3f5573-c264-4a8b-a2f0-0e6473d39aad"
+          (reference "R13") (unit 1)
+        )
+      )
+    )
+  )
   (symbol (lib_id "Connector_Generic:Conn_01x06") (at 267.97 109.22 0) (unit 1)
     (in_bom yes) (on_board yes) (dnp no) (fields_autoplaced)
@@
         )
       )
+    )
+  )
+  (symbol (lib_id "Device:R_Small") (at 236.22 82.55 270) (unit 1)
+    (in_bom yes) (on_board yes) (dnp no)
+    (property "Reference" "R14" (at 229.87 81.28 90)
+      (effects (font (size 1.27 1.27)) (justify left))
+    )
+    (property "Value" "4.7K" (at 234.8475 82.5656 90)
+      (effects (font (size 0.8 0.8)) (justify left))
+    )
+    (property "Footprint" "Resistor_SMD:R_0603_1608Metric" (at 236.22 82.55 0)
+      (effects (font (size 1.27 1.27)) hide)
+    )
+    (property "Datasheet" "~" (at 236.22 82.55 0)
+      (effects (font (size 1.27 1.27)) hide)
+    )
+    (property "LCSC" "C23186" (at 236.22 82.55 0)
+      (effects (font (size 1.27 1.27)) hide)
+    )
+    (pin "1")
+    (pin "2")
+    (instances
+      (project "chu_arcade"
+        (path "/2e3f5573-c264-4a8b-a2f0-0e6473d39aad"
+          (reference "R14") (unit 1)
+        )
+      )
